File: kicad/cluster.sch (KiCad schematic (older format))
At the start: 16 parts, among them J1 Conn_01x07, Q1 PT908-7B-F, Q2 PT908-7B-F, Q3 PT908-7B-F, Q4 PT908-7B-F, Q5 PT908-7B-F

Commit message: Update the names for the LEDs and PTs on the finger cluster pcb
Q -> PT
D -> IR
Parts:
- renumbered D1 to IR1, D2 to IR2, D3 to IR3, D4 to IR4, D5 to IR5, Q1 to PT1, Q2 to PT2, Q3 to PT3, Q4 to PT4, Q5 to PT5
Changed lines of the file:
@@
 $EndComp
 $Comp
-L lalboard:PT908-7B-F Q1
+L lalboard:PT908-7B-F PT1
 U 1 1 5F96F978
 P 5950 1750
-F 0 "Q1" H 6141 1796 50  0000 L CNN
+F 0 "PT1" H 6141 1796 50  0000 L CNN
 F 1 "PT908-7B-F" H 6141 1705 50  0000 L CNN
 F 2 "LED_THT:LED_SideEmitter_Rectangular_W4.5mm_H1.6mm" H 6430 1610 50  0001 C CNN
@@
 $EndComp
 $Comp
-L lalboard:IR908-7C-F D1
+L lalboard:IR908-7C-F IR1
 U 1 1 5F96F62E
 P 5450 1800
-F 0 "D1" V 5300 1700 50  0000 C CNN
+F 0 "IR1" V 5300 1700 50  0000 C CNN
 F 1 "IR908-7C-F" V 5400 1500 50  0000 C CNN
 F 2 "LED_THT:LED_SideEmitter_Rectangular_W4.5mm_H1.6mm" H 5450 1975 50  0001 C CNN
@@
 	5450 1400 5450 1600
 $Comp
-L lalboard:PT908-7B-F Q2
+L lalboard:PT908-7B-F PT2
 U 1 1 5F9B9EF8
 P 5950 2750
-F 0 "Q2" H 6141 2796 50  0000 L CNN
+F 0 "PT2" H 6141 2796 50  0000 L CNN
 F 1 "PT908-7B-F" H 6141 2705 50  0000 L CNN
 F 2 "LED_THT:LED_SideEmitter_Rectangular_W4.5mm_H1.6mm" H 6430 2610 50  0001 C CNN
@@
 $EndComp
 $Comp
-L lalboard:IR908-7C-F D2
+L lalboard:IR908-7C-F IR2
 U 1 1 5F9B9F04
 P 5450 2800
-F 0 "D2" V 5300 2700 50  0000 C CNN
+F 0 "IR2" V 5300 2700 50  0000 C CNN
 F 1 "IR908-7C-F" V 5400 2500 50  0000 C CNN
 F 2 "LED_THT:LED_SideEmitter_Rectangular_W4.5mm_H1.6mm" H 5450 2975 50  0001 C CNN
@@
 	5450 2400 5450 2600
 $Comp
-L lalboard:PT908-7B-F Q3
+L lalboard:PT908-7B-F PT3
 U 1 1 5F9BC92B
 P 5950 3750
-F 0 "Q3" H 6141 3796 50  0000 L CNN
+F 0 "PT3" H 6141 3796 50  0000 L CNN
 F 1 "PT908-7B-F" H 6141 3705 50  0000 L CNN
 F 2 "LED_THT:LED_SideEmitter_Rectangular_W4.5mm_H1.6mm" H 6430 3610 50  0001 C CNN
@@
 $EndComp
 $Comp
-L lalboard:IR908-7C-F D3
+L lalboard:IR908-7C-F IR3
 U 1 1 5F9BC937
 P 5450 3800
-F 0 "D3" V 5300 3700 50  0000 C CNN
+F 0 "IR3" V 5300 3700 50  0000 C CNN
 F 1 "IR908-7C-F" V 5400 3500 50  0000 C CNN
 F 2 "LED_THT:LED_SideEmitter_Rectangular_W4.5mm_H1.6mm" H 5450 3975 50  0001 C CNN
@@
 	5450 3400 5450 3600
 $Comp
-L lalboard:PT908-7B-F Q4
+L lalboard:PT908-7B-F PT4
 U 1 1 5F9BE283
 P 5950 4700
-F 0 "Q4" H 6141 4746 50  0000 L CNN
+F 0 "PT4" H 6141 4746 50  0000 L CNN
 F 1 "PT908-7B-F" H 6141 4655 50  0000 L CNN
 F 2 "LED_THT:LED_SideEmitter_Rectangular_W4.5mm_H1.6mm" H 6430 4560 50  0001 C CNN
@@
 $EndComp
 $Comp
-L lalboard:IR908-7C-F D4
+L lalboard:IR908-7C-F IR4
 U 1 1 5F9BE28F
 P 5450 4750
-F 0 "D4" V 5300 4650 50  0000 C CNN
+F 0 "IR4" V 5300 4650 50  0000 C CNN
 F 1 "IR908-7C-F" V 5400 4450 50  0000 C CNN
 F 2 "LED_THT:LED_SideEmitter_Rectangular_W4.5mm_H1.6mm" H 5450 4925 50  0001 C CNN
@@
 	5450 4350 5450 4550
 $Comp
-L lalboard:PT908-7B-F Q5
+L lalboard:PT908-7B-F PT5
 U 1 1 5F9BF567
 P 5950 5750
-F 0 "Q5" H 6141 5796 50  0000 L CNN
+F 0 "PT5" H 6141 5796 50  0000 L CNN
 F 1 "PT908-7B-F" H 6141 5705 50  0000 L CNN
 F 2 "LED_THT:LED_SideEmitter_Rectangular_W4.5mm_H1.6mm" H 6430 5610 50  0001 C CNN
@@
 $EndComp
 $Comp
-L lalboard:IR908-7C-F D5
+L lalboard:IR908-7C-F IR5
 U 1 1 5F9BF573
 P 5450 5800
-F 0 "D5" V 5300 5700 50  0000 C CNN
+F 0 "IR5" V 5300 5700 50  0000 C CNN
 F 1 "IR908-7C-F" V 5400 5500 50  0000 C CNN
 F 2 "LED_THT:LED_SideEmitter_Rectangular_W4.5mm_H1.6mm" H 5450 5975 50  0001 C CNN

Commit message: Add a nub indicating the lens on the IR and PT footprints
Parts:
- IR1, IR2, IR3, IR4, IR5: footprint LED_THT:LED_SideEmitter_Rectangular_W4.5mm_H1.6mm -> lalboard:IR908-7C-F
- PT1, PT2, PT3, PT4, PT5: footprint LED_THT:LED_SideEmitter_Rectangular_W4.5mm_H1.6mm -> lalboard:PT908-7C-F
Changed lines of the file:
@@
 F 0 "PT1" H 6141 1796 50  0000 L CNN
 F 1 "PT908-7B-F" H 6141 1705 50  0000 L CNN
-F 2 "LED_THT:LED_SideEmitter_Rectangular_W4.5mm_H1.6mm" H 6430 1610 50  0001 C CNN
+F 2 "lalboard:PT908-7C-F" H 6430 1610 50  0001 C CNN
 F 3 "https://www.everlight.com/file/ProductFile/PT908-7B-F.pdf" H 5950 1750 50  0001 C CNN
 	1    5950 1750
@@
 F 0 "IR1" V 5300 1700 50  0000 C CNN
 F 1 "IR908-7C-F" V 5400 1500 50  0000 C CNN
-F 2 "LED_THT:LED_SideEmitter_Rectangular_W4.5mm_H1.6mm" H 5450 1975 50  0001 C CNN
+F 2 "lalboard:IR908-7C-F" H 5450 1975 50  0001 C CNN
 F 3 "https://www.everlight.com/file/ProductFile/201407052136280483.pdf" H 5400 1800 50  0001 C CNN
 	1    5450 1800
@@
 F 0 "PT2" H 6141 2796 50  0000 L CNN
 F 1 "PT908-7B-F" H 6141 2705 50  0000 L CNN
-F 2 "LED_THT:LED_SideEmitter_Rectangular_W4.5mm_H1.6mm" H 6430 2610 50  0001 C CNN
+F 2 "lalboard:PT908-7C-F" H 6430 2610 50  0001 C CNN
 F 3 "https://www.everlight.com/file/ProductFile/PT908-7B-F.pdf" H 5950 2750 50  0001 C CNN
 	1    5950 2750
@@
 F 0 "IR2" V 5300 2700 50  0000 C CNN
 F 1 "IR908-7C-F" V 5400 2500 50  0000 C CNN
-F 2 "LED_THT:LED_SideEmitter_Rectangular_W4.5mm_H1.6mm" H 5450 2975 50  0001 C CNN
+F 2 "lalboard:IR908-7C-F" H 5450 2975 50  0001 C CNN
 F 3 "https://www.everlight.com/file/ProductFile/201407052136280483.pdf" H 5400 2800 50  0001 C CNN
 	1    5450 2800
@@
 F 0 "PT3" H 6141 3796 50  0000 L CNN
 F 1 "PT908-7B-F" H 6141 3705 50  0000 L CNN
-F 2 "LED_THT:LED_SideEmitter_Rectangular_W4.5mm_H1.6mm" H 6430 3610 50  0001 C CNN
+F 2 "lalboard:PT908-7C-F" H 6430 3610 50  0001 C CNN
 F 3 "https://www.everlight.com/file/ProductFile/PT908-7B-F.pdf" H 5950 3750 50  0001 C CNN
 	1    5950 3750
@@
 F 0 "IR3" V 5300 3700 50  0000 C CNN
 F 1 "IR908-7C-F" V 5400 3500 50  0000 C CNN
-F 2 "LED_THT:LED_SideEmitter_Rectangular_W4.5mm_H1.6mm" H 5450 3975 50  0001 C CNN
+F 2 "lalboard:IR908-7C-F" H 5450 3975 50  0001 C CNN
 F 3 "https://www.everlight.com/file/ProductFile/201407052136280483.pdf" H 5400 3800 50  0001 C CNN
 	1    5450 3800
@@
 F 0 "PT4" H 6141 4746 50  0000 L CNN
 F 1 "PT908-7B-F" H 6141 4655 50  0000 L CNN
-F 2 "LED_THT:LED_SideEmitter_Rectangular_W4.5mm_H1.6mm" H 6430 4560 50  0001 C CNN
+F 2 "lalboard:PT908-7C-F" H 6430 4560 50  0001 C CNN
 F 3 "https://www.everlight.com/file/ProductFile/PT908-7B-F.pdf" H 5950 4700 50  0001 C CNN
 	1    5950 4700
@@
 F 0 "IR4" V 5300 4650 50  0000 C CNN
 F 1 "IR908-7C-F" V 5400 4450 50  0000 C CNN
-F 2 "LED_THT:LED_SideEmitter_Rectangular_W4.5mm_H1.6mm" H 5450 4925 50  0001 C CNN
+F 2 "lalboard:IR908-7C-F" H 5450 4925 50  0001 C CNN
 F 3 "https://www.everlight.com/file/ProductFile/201407052136280483.pdf" H 5400 4750 50  0001 C CNN
 	1    5450 4750
@@
 F 0 "PT5" H 6141 5796 50  0000 L CNN
 F 1 "PT908-7B-F" H 6141 5705 50  0000 L CNN
-F 2 "LED_THT:LED_SideEmitter_Rectangular_W4.5mm_H1.6mm" H 6430 5610 50  0001 C CNN
+F 2 "lalboard:PT908-7C-F" H 6430 5610 50  0001 C CNN
 F 3 "https://www.everlight.com/file/ProductFile/PT908-7B-F.pdf" H 5950 5750 50  0001 C CNN
 	1    5950 5750
@@
 F 0 "IR5" V 5300 5700 50  0000 C CNN
 F 1 "IR908-7C-F" V 5400 5500 50  0000 C CNN
-F 2 "LED_THT:LED_SideEmitter_Rectangular_W4.5mm_H1.6mm" H 5450 5975 50  0001 C CNN
+F 2 "lalboard:IR908-7C-F" H 5450 5975 50  0001 C CNN
 F 3 "https://www.everlight.com/file/ProductFile/201407052136280483.pdf" H 5400 5800 50  0001 C CNN
 	1    5450 5800

Commit message: Update the kicad design for the finger cluster
This brings the PCB design up to par with the current cluster design.
Parts:
- J1: footprint lalboard:JST_ZH_B7B-ZR_1x07_P1.50mm_Vertical -> lalboard:JST_ZH_S7B-ZR_1x07_P1.50mm_Horizontal
Changed lines of the file:
@@
 F 0 "J1" H 3818 3375 50  0000 C CNN
 F 1 "Conn_01x07" H 3818 3466 50  0000 C CNN
-F 2 "lalboard:JST_ZH_B7B-ZR_1x07_P1.50mm_Vertical" H 3900 3900 50  0001 C CNN
+F 2 "lalboard:JST_ZH_S7B-ZR_1x07_P1.50mm_Horizontal" H 3900 3900 50  0001 C CNN
 F 3 "~" H 3900 3900 50  0001 C CNN
 	1    3900 3900

Commit message: Update kicad design for finger cluster
This adds ground/+5v planes, some thicker traces, and moves the +5v pin
to pin 1 of the connector.

Thanks to @rutgervana for taking a look at the design and making
suggestions/showing example improvements.
Connections:
- net labels added: C2
- net labels removed: C6
- wire segments 10 -> 0
Other:
- moved on the sheet: J1, R1

Commit message: Update the various sensitivity-related resistor values
This updates the transimpedance amplifier resistors to 2k, and adjusts
the LED drive resistors to an appropriate level, from empirical testing.
Parts:
- R1, R2, R3, R4, R5: value 150 -> 270
Other:
- note added: "Down"
- note added: "North"
- note added: "South"
- note added: "West"
Changed lines of the file:
@@
 P 3300 1550
 F 0 "R1" V 3400 1500 50  0000 L CNN
-F 1 "150" V 3294 1474 50  0000 L CNN
+F 1 "270" V 3294 1474 50  0000 L CNN
 F 2 "Resistor_SMD:R_1206_3216Metric_Pad1.42x1.75mm_HandSolder" V 3230 1550 50  0001 C CNN
 F 3 "~" H 3300 1550 50  0001 C CNN
@@
 P 3300 2850
 F 0 "R2" V 3400 2800 50  0000 L CNN
-F 1 "150" V 3294 2774 50  0000 L CNN
+F 1 "270" V 3294 2774 50  0000 L CNN
 F 2 "Resistor_SMD:R_1206_3216Metric_Pad1.42x1.75mm_HandSolder" V 3230 2850 50  0001 C CNN
 F 3 "~" H 3300 2850 50  0001 C CNN
@@
 P 3300 4150
 F 0 "R3" V 3400 4100 50  0000 L CNN
-F 1 "150" V 3294 4074 50  0000 L CNN
+F 1 "270" V 3294 4074 50  0000 L CNN
 F 2 "Resistor_SMD:R_1206_3216Metric_Pad1.42x1.75mm_HandSolder" V 3230 4150 50  0001 C CNN
 F 3 "~" H 3300 4150 50  0001 C CNN
@@
 P 3300 5450
 F 0 "R4" V 3400 5400 50  0000 L CNN
-F 1 "150" V 3294 5374 50  0000 L CNN
+F 1 "270" V 3294 5374 50  0000 L CNN
 F 2 "Resistor_SMD:R_1206_3216Metric_Pad1.42x1.75mm_HandSolder" V 3230 5450 50  0001 C CNN
 F 3 "~" H 3300 5450 50  0001 C CNN
@@
 P 3300 6750
 F 0 "R5" V 3400 6700 50  0000 L CNN
-F 1 "150" V 3294 6674 50  0000 L CNN
+F 1 "270" V 3294 6674 50  0000 L CNN
 F 2 "Resistor_SMD:R_1206_3216Metric_Pad1.42x1.75mm_HandSolder" V 3230 6750 50  0001 C CNN
 F 3 "~" H 3300 6750 50  0001 C CNN
@@
 Wire Notes Line
 	3050 6000 3050 7200
+Text Notes 3850 4550 0    50   ~ 0
+Down
+Text Notes 3900 1950 0    50   ~ 0
+West
+Text Notes 3850 3250 0    50   ~ 0
+South
+Text Notes 3850 5850 0    50   ~ 0
+North
+Text Notes 3850 7150 0    50   ~ 0
+South
 $EndSCHEMATC
