File: kicad/thumb_cluster_left.sch (KiCad schematic (older format))
At the start: 16 parts, among them J1 Conn_01x07

Commit message: Update the design of the left thumb cluster pcb
Parts:
- R1: value 150 -> 100
Connections:
- net labels added: C2
- net labels removed: C6
- wire segments 10 -> 0
Other:
- moved on the sheet: J1, R1

Commit message: Update thumb cluster pcbs to v0.2
This shuffles the switch numbering and order on the connector,
so that the center key is on the same pin of the connector (pin 4)
as the center key of the finger clusters.

These keys on the thumb and finger clusters have inverted logic from
all the other keys, due to the physical design of the switches. This
puts the inverted keys on the same pin/column. This simplifies the
firmware a bit, because it can just assume that pin is always inverted.
Parts:
- added H1, H2: MountingHole_Pad, MountingHole:MountingHole_3.2mm_M3_Pad, symbol Mechanical:MountingHole_Pad
Changed lines of the file:
@@
 Wire Notes Line
 	3050 6000 3050 7200
+$Comp
+L Mechanical:MountingHole_Pad H1
+U 1 1 60869011
+P 1350 7150
+F 0 "H1" H 1250 7200 50  0000 R CNN
+F 1 "MountingHole_Pad" H 1250 7100 50  0000 R CNN
+F 2 "MountingHole:MountingHole_3.2mm_M3_Pad" H 1350 7150 50  0001 C CNN
+F 3 "~" H 1350 7150 50  0001 C CNN
+	1    1350 7150
+	1    0    0    -1
+$EndComp
+$Comp
+L Mechanical:MountingHole_Pad H2
+U 1 1 6086CECE
+P 1550 7150
+F 0 "H2" H 1650 7199 50  0000 L CNN
+F 1 "MountingHole_Pad" H 1650 7108 50  0000 L CNN
+F 2 "MountingHole:MountingHole_3.2mm_M3_Pad" H 1550 7150 50  0001 C CNN
+F 3 "~" H 1550 7150 50  0001 C CNN
+	1    1550 7150
+	1    0    0    -1
+$EndComp
+$Comp
+L power:GND #PWR0113
+U 1 1 6086D422
+P 1350 7250
+F 0 "#PWR0113" H 1350 7000 50  0001 C CNN
+F 1 "GND" H 1355 7077 50  0000 C CNN
+F 2 "" H 1350 7250 50  0001 C CNN
+F 3 "" H 1350 7250 50  0001 C CNN
+	1    1350 7250
+	1    0    0    -1
+$EndComp
+$Comp
+L power:GND #PWR0114
+U 1 1 6086D6EB
+P 1550 7250
+F 0 "#PWR0114" H 1550 7000 50  0001 C CNN
+F 1 "GND" H 1555 7077 50  0000 C CNN
+F 2 "" H 1550 7250 50  0001 C CNN
+F 3 "" H 1550 7250 50  0001 C CNN
+	1    1550 7250
+	1    0    0    -1
+$EndComp
 $EndSCHEMATC

Commit message: Update the various sensitivity-related resistor values
This updates the transimpedance amplifier resistors to 2k, and adjusts
the LED drive resistors to an appropriate level, from empirical testing.
Parts:
- R1: value 100 -> 56
- R2: value 150 -> 100
- R3: value 150 -> 120
- R4: value 150 -> 180
Other:
- note added: "Down"
- note added: "Inner"
- note added: "Lower Outer"
- note added: "Mode"
- note added: "Upper Outer"
Changed lines of the file:
@@
 C5
-$Comp
-L Device:R R1
-U 1 1 5F993655
-P 3300 1550
-F 0 "R1" V 3400 1500 50  0000 L CNN
-F 1 "100" V 3294 1474 50  0000 L CNN
-F 2 "Resistor_SMD:R_1206_3216Metric_Pad1.42x1.75mm_HandSolder" V 3230 1550 50  0001 C CNN
-F 3 "~" H 3300 1550 50  0001 C CNN
-	1    3300 1550
-	-1   0    0    1
-$EndComp
 $Comp
 L lalboard:IR908-7C-F IR1
@@
 P 3300 2850
 F 0 "R2" V 3400 2800 50  0000 L CNN
-F 1 "150" V 3294 2774 50  0000 L CNN
+F 1 "100" V 3294 2774 50  0000 L CNN
 F 2 "Resistor_SMD:R_1206_3216Metric_Pad1.42x1.75mm_HandSolder" V 3230 2850 50  0001 C CNN
 F 3 "~" H 3300 2850 50  0001 C CNN
@@
 P 3300 4150
 F 0 "R3" V 3400 4100 50  0000 L CNN
-F 1 "150" V 3294 4074 50  0000 L CNN
+F 1 "120" V 3294 4074 50  0000 L CNN
 F 2 "Resistor_SMD:R_1206_3216Metric_Pad1.42x1.75mm_HandSolder" V 3230 4150 50  0001 C CNN
 F 3 "~" H 3300 4150 50  0001 C CNN
@@
 P 3300 5450
 F 0 "R4" V 3400 5400 50  0000 L CNN
-F 1 "150" V 3294 5374 50  0000 L CNN
+F 1 "180" V 3294 5374 50  0000 L CNN
 F 2 "Resistor_SMD:R_1206_3216Metric_Pad1.42x1.75mm_HandSolder" V 3230 5450 50  0001 C CNN
 F 3 "~" H 3300 5450 50  0001 C CNN
@@
 	1    0    0    -1
 $EndComp
+Text Notes 3600 3250 0    50   ~ 0
+Upper Outer
+Text Notes 3600 1950 0    50   ~ 0
+Lower Outer
+Text Notes 3850 4550 0    50   ~ 0
+Down
+Text Notes 3850 5850 0    50   ~ 0
+Inner
+Text Notes 3850 7150 0    50   ~ 0
+Mode
+$Comp
+L Device:R R1
+U 1 1 5F993655
+P 3300 1550
+F 0 "R1" V 3400 1500 50  0000 L CNN
+F 1 "56" V 3294 1474 50  0000 L CNN
+F 2 "Resistor_SMD:R_1206_3216Metric_Pad1.42x1.75mm_HandSolder" V 3230 1550 50  0001 C CNN
+F 3 "~" H 3300 1550 50  0001 C CNN
+	1    3300 1550
+	-1   0    0    1
+$EndComp
 $EndSCHEMATC
